Commit message: done modelling all links and joint

File: urdf/pivot.urdf.xacro (robot description, xacro)
@@ -2,4 +2,5 @@
 <robot name="atm" xmlns:xacro="http://ros.org/wiki/xacro">
   <link name="base_footprint"/>
+<!-- base link n joint-->
     <link name="base_link">
     <visual>
@@ -8,6 +9,6 @@
         <mesh filename="package://pivot_description/meshes/base_link.stl" />
       </geometry>
-     <material name="green">
-        <color rgba="0.0 1.0 0.0 1.0"/>
+     <material name="chrome">
+        <color rgba="0.88 0.90 0.93 1.0"/>
      </material>
     </visual>
@@ -18,4 +19,5 @@
     <origin xyz="0 0 0.032" rpy="0 0 0"/>
   </joint>
+<!-- right wheel n joint-->
   <link name="right_wheel_link">
     <visual>
@@ -41,4 +43,5 @@
     <axis xyz="1 0 0" />
   </joint>
+  <!-- left wheel n joint-->
   <link
     name="left_wheel_link">
@@ -65,3 +68,123 @@
     <axis xyz="1 0 0" />
   </joint>
+  <!-- lidar n joint-->
+  <link
+    name="lidar_link">
+    <visual>
+      <origin xyz="0 0 0" rpy="0 0 0" />
+      <geometry>
+        <mesh filename="package://pivot_description/meshes/lidar_link.stl" />
+      </geometry>
+                 <material name="black">
+        <color rgba="0.0 0.0 0.0 1.0"/>
+     </material>
+    </visual>
+    <!--<collision>
+      <origin xyz="0 0.015 0" rpy="-1.57 0 0" />
+      <geometry>
+        <sphere radius="0.033"/>
+      </geometry>
+    </collision>-->
+  </link>
+  <joint name="lidar_joint" type="fixed">
+    <origin xyz="0 0 0.18515" rpy="0 0 0" />
+    <parent link="base_link" />
+    <child link="lidar_link" />
+  </joint>
+ <!-- camera n joint-->
+  <link
+    name="camera_link">
+    <visual>
+      <origin xyz="0 0 0" rpy="0 0 0" />
+      <geometry>
+        <mesh filename="package://pivot_description/meshes/camera_link.stl" />
+      </geometry>
+                 <material name="black">
+        <color rgba="0.0 0.0 0.0 1.0"/>
+     </material>
+    </visual>
+    <!--<collision>
+      <origin xyz="0 0.015 0" rpy="-1.57 0 0" />
+      <geometry>
+        <sphere radius="0.033"/>
+      </geometry>
+    </collision>-->
+  </link>
+  <joint name="camera_joint" type="fixed">
+    <origin xyz="-0.0045 -0.11826 0.13872" rpy="0 0 0" />
+    <parent link="base_link" />
+    <child link="camera_link" />
+  </joint>
+  <!-- front_sonic n joint-->
+  <link
+    name="ultrasonic_front_link">
+    <visual>
+      <origin xyz="0 0 0" rpy="0 0 0" />
+      <geometry>
+        <mesh filename="package://pivot_description/meshes/front_sonic_link.stl" />
+      </geometry>
+                 <material name="pcb_green">
+        <color rgba="0.06 0.35 0.18 1.0"/>
+     </material>
+    </visual>
+    <!--<collision>
+      <origin xyz="0 0.015 0" rpy="-1.57 0 0" />
+      <geometry>
+        <sphere radius="0.033"/>
+      </geometry>
+    </collision>-->
+  </link>
+  <joint name="ultrasonic_front_joint" type="fixed">
+    <origin xyz="0 -0.06698 0.0645" rpy="0 0 0" />
+    <parent link="base_link" />
+    <child link="ultrasonic_front_link" />
+  </joint>
+  <!-- right_sonic n joint-->
+  <link
+    name="ultrasonic_right_link">
+    <visual>
+      <origin xyz="0 0 0" rpy="0 0 0" />
+      <geometry>
+        <mesh filename="package://pivot_description/meshes/right_sonic_link.stl" />
+      </geometry>
+                 <material name="pcb_green">
+        <color rgba="0.06 0.35 0.18 1.0"/>
+     </material>
+    </visual>
+    <!--<collision>
+      <origin xyz="0 0.015 0" rpy="-1.57 0 0" />
+      <geometry>
+        <sphere radius="0.033"/>
+      </geometry>
+    </collision>-->
+  </link>
+  <joint name="ultrasonic_right_joint" type="fixed">
+    <origin xyz="-0.05245 0 0.0657" rpy="0 0 0" />
+    <parent link="base_link" />
+    <child link="ultrasonic_right_link" />
+  </joint>
+  <!-- left_sonic n joint-->
+  <link
+    name="ultrasonic_left_link">
+    <visual>
+      <origin xyz="0 0 0" rpy="0 0 0" />
+      <geometry>
+        <mesh filename="package://pivot_description/meshes/left_sonic_link.stl" />
+      </geometry>
+                 <material name="pcb_green">
+        <color rgba="0.06 0.35 0.18 1.0"/>
+     </material>
+    </visual>
+    <!--<collision>
+      <origin xyz="0 0.015 0" rpy="-1.57 0 0" />
+      <geometry>
+        <sphere radius="0.033"/>
+      </geometry>
+    </collision>-->
+  </link>
+  <joint name="ultrasonic_left_joint" type="fixed">
+    <origin xyz="0.05245 0 0.0657" rpy="0 0 0" />
+    <parent link="base_link" />
+    <child link="ultrasonic_left_link" />
+  </joint>
   </robot>

Commit message: fixed lidar pos and robot orientation

File: urdf/pivot.urdf.xacro (robot description, xacro)
@@ -1,9 +1,9 @@
 <?xml version="1.0" encoding="UTF-8"?>
-<robot name="atm" xmlns:xacro="http://ros.org/wiki/xacro">
+<robot name="pivot" xmlns:xacro="http://www.ros.org/wiki/xacro">
   <link name="base_footprint"/>
 <!-- base link n joint-->
     <link name="base_link">
     <visual>
-      <origin xyz="0 0 0" rpy="0 0 0" />
+      <origin xyz="0 0 0" rpy="0 0 1.5708" />
       <geometry>
         <mesh filename="package://pivot_description/meshes/base_link.stl" />
@@ -17,10 +17,10 @@
     <parent link="base_footprint"/>
     <child link="base_link" />
-    <origin xyz="0 0 0.032" rpy="0 0 0"/>
+    <origin xyz="0 0 0.064" rpy="0 0 0"/>
   </joint>
 <!-- right wheel n joint-->
   <link name="right_wheel_link">
     <visual>
-      <origin xyz="0 0 0" rpy="0 0 0" />
+      <origin xyz="0 0 0" rpy="0 0 1.5708" />
       <geometry>
         <mesh filename="package://pivot_description/meshes/right_wheel_link.stl" />
@@ -38,8 +38,8 @@
   </link>
   <joint name="right_wheel_joint" type="continuous">
-    <origin xyz="-0.079 0 -0.0305" rpy="0 0 0" />
+    <origin xyz="0 -0.079 -0.0305" rpy="0 0 0" />
     <parent link="base_link" />
     <child link="right_wheel_link" />
-    <axis xyz="1 0 0" />
+    <axis xyz="0 1 0" />
   </joint>
   <!-- left wheel n joint-->
@@ -47,5 +47,5 @@
     name="left_wheel_link">
     <visual>
-      <origin xyz="0 0 0" rpy="0 0 0" />
+      <origin xyz="0 0 0" rpy="0 0 1.5708" />
       <geometry>
         <mesh filename="package://pivot_description/meshes/left_wheel_link.stl" />
@@ -63,8 +63,8 @@
   </link>
   <joint name="left_wheel_joint" type="continuous">
-    <origin xyz="0.079 0 -0.0305" rpy="0 0 0" />
+    <origin xyz="0 0.079 -0.0305" rpy="0 0 0" />
     <parent link="base_link" />
     <child link="left_wheel_link" />
-    <axis xyz="1 0 0" />
+    <axis xyz="0 1 0" />
   </joint>
   <!-- lidar n joint-->
@@ -72,5 +72,5 @@
     name="lidar_link">
     <visual>
-      <origin xyz="0 0 0" rpy="0 0 0" />
+      <origin xyz="0 0 0" rpy="0 0 1.5708" />
       <geometry>
         <mesh filename="package://pivot_description/meshes/lidar_link.stl" />
@@ -88,5 +88,5 @@
   </link>
   <joint name="lidar_joint" type="fixed">
-    <origin xyz="0 0 0.18515" rpy="0 0 0" />
+    <origin xyz="0.00079 -0.0014 0.18515" rpy="0 0 0" />
     <parent link="base_link" />
     <child link="lidar_link" />
@@ -96,5 +96,5 @@
     name="camera_link">
     <visual>
-      <origin xyz="0 0 0" rpy="0 0 0" />
+      <origin xyz="0 0 0" rpy="0 0 1.5708" />
       <geometry>
         <mesh filename="package://pivot_description/meshes/camera_link.stl" />
@@ -112,5 +112,5 @@
   </link>
   <joint name="camera_joint" type="fixed">
-    <origin xyz="-0.0045 -0.11826 0.13872" rpy="0 0 0" />
+    <origin xyz="0.11826 -0.0045 0.13872" rpy="0 0 0" />
     <parent link="base_link" />
     <child link="camera_link" />
@@ -120,5 +120,5 @@
     name="ultrasonic_front_link">
     <visual>
-      <origin xyz="0 0 0" rpy="0 0 0" />
+      <origin xyz="0 0 0" rpy="0 0 1.5708" />
       <geometry>
         <mesh filename="package://pivot_description/meshes/front_sonic_link.stl" />
@@ -136,5 +136,5 @@
   </link>
   <joint name="ultrasonic_front_joint" type="fixed">
-    <origin xyz="0 -0.06698 0.0645" rpy="0 0 0" />
+    <origin xyz="0.06698 0 0.0645" rpy="0 0 0" />
     <parent link="base_link" />
     <child link="ultrasonic_front_link" />
@@ -144,5 +144,5 @@
     name="ultrasonic_right_link">
     <visual>
-      <origin xyz="0 0 0" rpy="0 0 0" />
+      <origin xyz="0 0 0" rpy="0 0 1.5708" />
       <geometry>
         <mesh filename="package://pivot_description/meshes/right_sonic_link.stl" />
@@ -160,5 +160,5 @@
   </link>
   <joint name="ultrasonic_right_joint" type="fixed">
-    <origin xyz="-0.05245 0 0.0657" rpy="0 0 0" />
+    <origin xyz="0 -0.05245 0.0657" rpy="0 0 0" />
     <parent link="base_link" />
     <child link="ultrasonic_right_link" />
@@ -168,5 +168,5 @@
     name="ultrasonic_left_link">
     <visual>
-      <origin xyz="0 0 0" rpy="0 0 0" />
+      <origin xyz="0 0 0" rpy="0 0 1.5708" />
       <geometry>
         <mesh filename="package://pivot_description/meshes/left_sonic_link.stl" />
@@ -184,5 +184,5 @@
   </link>
   <joint name="ultrasonic_left_joint" type="fixed">
-    <origin xyz="0.05245 0 0.0657" rpy="0 0 0" />
+    <origin xyz="0 0.05245 0.0657" rpy="0 0 0" />
     <parent link="base_link" />
     <child link="ultrasonic_left_link" />

Commit message: Add Gazebo simulation support

File: urdf/pivot.urdf.xacro (robot description, xacro)
@@ -1,4 +1,5 @@
 <?xml version="1.0" encoding="UTF-8"?>
 <robot name="pivot" xmlns:xacro="http://www.ros.org/wiki/xacro">
+  <xacro:include filename="$(find pivot_description)/urdf/pivot_gazebo.xacro"/>
   <link name="base_footprint"/>
 <!-- base link n joint-->
@@ -13,4 +14,16 @@
      </material>
     </visual>
+        <inertial>
+      <origin xyz="0 0 0.0583" rpy="0 0 0"/>
+      <mass value="1.225"/>
+      <inertia ixx="0.00699" iyy="0.00657" izz="0.00227"
+               ixy="0" ixz="0" iyz="0"/>
+    </inertial>
+    <collision>
+  <origin xyz="0 0 0.0895" rpy="0 0 0" />
+<geometry>
+  <box size="0.14128 0.120 0.217"/>
+</geometry>
+</collision>
   </link>
   <joint name="base_joint" type="fixed">
@@ -30,10 +43,16 @@
      </material>
     </visual>
-    <!--<collision>
-      <origin xyz="0 -0.015 0" rpy="1.57 0 0" />
-      <geometry>
-        <sphere radius="0.033"/>
-      </geometry>
-    </collision>-->
+        <inertial>
+      <origin xyz="0 0 0" rpy="0 0 0"/>
+      <mass value="0.0988"/>
+      <inertia ixx="3.74e-5" iyy="6.60e-5" izz="3.74e-5"
+               ixy="0" ixz="0" iyz="0"/>
+    </inertial>
+    <collision>
+      <origin xyz="0 0 0" rpy="1.5708 0 0" />
+      <geometry>
+        <cylinder radius="0.0335" length="0.027"/>
+      </geometry>
+    </collision>
   </link>
   <joint name="right_wheel_joint" type="continuous">
@@ -42,4 +61,5 @@
     <child link="right_wheel_link" />
     <axis xyz="0 1 0" />
+        <dynamics damping="0.01" friction="0.001"/>
   </joint>
   <!-- left wheel n joint-->
@@ -55,10 +75,16 @@
      </material>
     </visual>
-    <!--<collision>
-      <origin xyz="0 0.015 0" rpy="-1.57 0 0" />
-      <geometry>
-        <sphere radius="0.033"/>
-      </geometry>
-    </collision>-->
+        <inertial>
+      <origin xyz="0 0 0" rpy="0 0 0"/>
+      <mass value="0.0988"/>
+      <inertia ixx="3.74e-5" iyy="6.60e-5" izz="3.74e-5"
+               ixy="0" ixz="0" iyz="0"/>
+    </inertial>
+    <collision>
+      <origin xyz="0 0 0" rpy="1.5708 0 0" />
+      <geometry>
+        <cylinder radius="0.0335" length="0.027"/>
+      </geometry>
+    </collision>
   </link>
   <joint name="left_wheel_joint" type="continuous">
@@ -67,4 +93,19 @@
     <child link="left_wheel_link" />
     <axis xyz="0 1 0" />
+        <dynamics damping="0.01" friction="0.001"/>
+  </joint>
+     <!-- imu n joint-->
+  <link name="imu_link">
+    <inertial>
+      <origin xyz="0 0 0" rpy="0 0 0"/>
+      <mass value="1e-5"/>
+      <inertia ixx="1e-9" iyy="1e-9" izz="1e-9"
+               ixy="0" ixz="0" iyz="0"/>
+    </inertial>
+  </link>
+  <joint name="imu_joint" type="fixed">
+    <origin xyz="0 0 0" rpy="0 0 0" />
+    <parent link="base_link" />
+    <child link="imu_link" />
   </joint>
   <!-- lidar n joint-->
@@ -80,10 +121,10 @@
      </material>
     </visual>
-    <!--<collision>
-      <origin xyz="0 0.015 0" rpy="-1.57 0 0" />
-      <geometry>
-        <sphere radius="0.033"/>
-      </geometry>
-    </collision>-->
+        <inertial>
+      <origin xyz="0 0 0" rpy="0 0 0"/>
+      <mass value="1e-5"/>
+      <inertia ixx="1e-9" iyy="1e-9" izz="1e-9"
+               ixy="0" ixz="0" iyz="0"/>
+    </inertial>
   </link>
   <joint name="lidar_joint" type="fixed">
@@ -104,10 +145,10 @@
      </material>
     </visual>
-    <!--<collision>
-      <origin xyz="0 0.015 0" rpy="-1.57 0 0" />
-      <geometry>
-        <sphere radius="0.033"/>
-      </geometry>
-    </collision>-->
+        <inertial>
+      <origin xyz="0 0 0" rpy="0 0 0"/>
+      <mass value="1e-5"/>
+      <inertia ixx="1e-9" iyy="1e-9" izz="1e-9"
+               ixy="0" ixz="0" iyz="0"/>
+    </inertial>
   </link>
   <joint name="camera_joint" type="fixed">
@@ -128,10 +169,10 @@
      </material>
     </visual>
-    <!--<collision>
-      <origin xyz="0 0.015 0" rpy="-1.57 0 0" />
-      <geometry>
-        <sphere radius="0.033"/>
-      </geometry>
-    </collision>-->
+        <inertial>
+      <origin xyz="0 0 0" rpy="0 0 0"/>
+      <mass value="1e-5"/>
+      <inertia ixx="1e-9" iyy="1e-9" izz="1e-9"
+               ixy="0" ixz="0" iyz="0"/>
+    </inertial>
   </link>
   <joint name="ultrasonic_front_joint" type="fixed">
@@ -152,10 +193,10 @@
      </material>
     </visual>
-    <!--<collision>
-      <origin xyz="0 0.015 0" rpy="-1.57 0 0" />
-      <geometry>
-        <sphere radius="0.033"/>
-      </geometry>
-    </collision>-->
+        <inertial>
+      <origin xyz="0 0 0" rpy="0 0 0"/>
+      <mass value="1e-5"/>
+      <inertia ixx="1e-9" iyy="1e-9" izz="1e-9"
+               ixy="0" ixz="0" iyz="0"/>
+    </inertial>
   </link>
   <joint name="ultrasonic_right_joint" type="fixed">
@@ -176,10 +217,10 @@
      </material>
     </visual>
-    <!--<collision>
-      <origin xyz="0 0.015 0" rpy="-1.57 0 0" />
-      <geometry>
-        <sphere radius="0.033"/>
-      </geometry>
-    </collision>-->
+        <inertial>
+      <origin xyz="0 0 0" rpy="0 0 0"/>
+      <mass value="1e-5"/>
+      <inertia ixx="1e-9" iyy="1e-9" izz="1e-9"
+               ixy="0" ixz="0" iyz="0"/>
+    </inertial>
   </link>
   <joint name="ultrasonic_left_joint" type="fixed">
